File: hardware/65x-io-w65c22.kicad_sch (KiCad schematic)
At the start: 1 part

Commit message: Update KiCad project files to current version
Parts:
- gave numbers to parts that had none: 1
Changed lines of the file:
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@@
 (kicad_sch
-  (version 20231120)
-  (generator "eeschema")
-  (generator_version "8.0")
-  (paper "A4")
-  (title_block
-    (title "65x Bus VIA I/O Card (W65C22)")
-    (date "2026-01-05")
-    (rev "0.1")
-    (company "65x Bus Project")
-    (comment 1 "WDC W65C22 VIA Parallel I/O Card")
-    (comment 2 "160mm x 100mm Eurocard 3U")
-  )
-  (symbol
-    (lib_id "")
-    (at 0 0 0)
-    (unit 1)
-    (exclude_from_sim no)
-    (in_bom yes)
-    (on_board yes)
-    (dnp no)
-  )
-  (sheet_instances
-    (path "/"
-      (page "1")
-    )
-  )
+	(version 20250114)
+	(generator "eeschema")
+	(generator_version "9.0")
+	(paper "A4")
+	(title_block
+		(title "65x Bus VIA I/O Card (W65C22)")
+		(date "2026-01-05")
+		(rev "0.1")
+		(company "65x Bus Project")
+		(comment 1 "WDC W65C22 VIA Parallel I/O Card")
+		(comment 2 "160mm x 100mm Eurocard 3U")
+	)
+	(symbol
+		(lib_id "")
+		(at 0 0 0)
+		(unit 1)
+		(exclude_from_sim no)
+		(in_bom yes)
+		(on_board yes)
+		(dnp no)
+		(property "Reference" "U?"
+			(at 0 0 0)
+			(effects
+				(font
+					(size 1.27 1.27)
+				)
+			)
+		)
+		(property "Value" ""
+			(at 0 0 0)
+			(effects
+				(font
+					(size 1.27 1.27)
+				)
+			)
+		)
+		(property "Footprint" ""
+			(at 0 0 0)
+			(effects
+				(font
+					(size 1.27 1.27)
+				)
+			)
+		)
+		(property "Datasheet" ""
+			(at 0 0 0)
+			(effects
+				(font
+					(size 1.27 1.27)
+				)
+			)
+		)
+		(property "Description" ""
+			(at 0 0 0)
+			(effects
+				(font
+					(size 1.27 1.27)
+				)
+			)
+		)
+		(instances
+			(project "65x-io-w65c22"
+				(path "/00000000-0000-0000-0000-000000000001"
+					(reference "U?")
+					(unit 1)
+				)
+			)
+		)
+	)
+	(sheet_instances
+		(path "/"
+			(page "1")
+		)
+	)
+	(embedded_fonts no)
 )
